Commit message: upgrade

File: catkin/src/tutorials/testbot_description/urdf/oneMesh.urdf (robot description, URDF)
Before this commit: robot one_mesh, 2 links, 1 joints
Links:
- link base_link: geometry visual mesh filename=package://testbot_description/meshes/mecanum.dae

Commit message: upgrade

File: catkin/src/tutorials/testbot_description/urdf/oneMesh.urdf (robot description, URDF)
Before this commit: robot one_mesh, 2 links, 1 joints
Links:
- removed link base_laser
- removed link base_link
- added link base_robot; visual box size=2 1 0.1
- added link base_wheel_back_left; visual mesh filename=package://testbot_description/meshes/mecanum.dae
- added link base_wheel_front_right; visual mesh filename=package://testbot_description/meshes/mecanum.dae
Joints:
- removed joint base_link_to_base_joint
- added joint base_robot_to_base_wheel: type continuous, parent base_robot, child base_wheel_back_left, origin xyz=-0.8 1 0, axis 0 1 0
- added joint base_robot_to_base_wheel_front_right: type continuous, parent base_robot, child base_wheel_front_right, origin xyz=0.8 -1 0, axis 0 1 0
