Commit message: upgrade

File: catkin/src/tutorials/testbot_description/urdf/robot_model.urdf.xacro (robot description, xacro)
@@ -1,5 +1,6 @@
 <?xml version="1.0" encoding="UTF-8"?>
 <robot name="robot_model" xmlns:xacro="http://www.ros.org/wiki/xacro" >
-	<xacro:property name="right_wheel_mesh_path" value="package://testbot_description/meshes/mecanum.dae" />
+	<xacro:property name="right_wheel_mesh_path" value="package://testbot_description/meshes/mecanumFrontRight.dae" />
+	<xacro:property name="left_wheel_mesh_path" value="package://testbot_description/meshes/mecanumFrontLeft.dae" />
 	<xacro:property name="wheel_distance_x" value="0.8"/>
 	<xacro:property name="wheel_distance_y" value="1" />
@@ -9,7 +10,10 @@
 			<origin rpy="0 0 0" xyz="0 0 0" />
 			<geometry>
-				<box size="2 1 0.1" />
+				<box size="2 1 0.4" />
 			</geometry>
-		</visual>
+			<material name="my_white">
+				<color rgba="1 1 1 0.8"/>
+			</material>
+		</visual>5
 	</link>
 	<link name="base_wheel_back_left">
@@ -29,4 +33,20 @@
 		</visual>
 	</link>
+	<link name="base_wheel_front_left">
+		<visual>
+			<origin rpy="1.57075 0 0" xyz="0 0 0" />
+			<geometry>
+				<mesh filename="${left_wheel_mesh_path}" scale="10 10 10" />
+			</geometry>
+		</visual>
+	</link>
+	<link name="base_wheel_back_right">
+		<visual>
+			<origin rpy="-1.57075 0 0" xyz="0 0 0" />
+			<geometry>
+				<mesh filename="${left_wheel_mesh_path}" scale="10 10 10" />
+			</geometry>
+		</visual>
+	</link>
 	<joint name="base_robot_to_base_wheel" type="${wheel_kinematic_type}" >
 		<parent link="base_robot" />
@@ -41,3 +61,15 @@
 		<origin xyz="${wheel_distance_x} -${wheel_distance_y} 0" />
 	</joint>
+	<joint name="base_robot_to_base_wheel_front_left" type="${wheel_kinematic_type}" >
+		<parent link="base_robot" />
+		<child link="base_wheel_front_left" />
+		<axis xyz="0 1 0" />
+		<origin xyz="${wheel_distance_x} ${wheel_distance_y} 0" />
+	</joint>
+	<joint name="base_robot_to_base_wheel_back_right" type="${wheel_kinematic_type}" >
+		<parent link="base_robot" />
+		<child link="base_wheel_back_right" />
+		<axis xyz="0 1 0" />
+		<origin xyz="-${wheel_distance_x} -${wheel_distance_y} 0" />
+	</joint>
 </robot>

Commit message: upgrade

File: catkin/src/tutorials/testbot_description/urdf/robot_model.urdf.xacro (robot description, xacro)
@@ -6,4 +6,6 @@
 	<xacro:property name="wheel_distance_y" value="1" />
 	<xacro:property name="wheel_kinematic_type" value="fixed" />
+	<xacro:property name="hokuyo_mesh_path" value="package://testbot_description/meshes/hokuyo.dae" />
+	<xacro:property name="hokuyo_kinematic_type" value="fixed" />
 	<link name="base_robot">
 		<visual>
@@ -49,4 +51,12 @@
 		</visual>
 	</link>
+	<link name="hokuyo_laser">
+		<visual>
+			<origin rpy="0 0 0" xyz="0 0 0" />
+			<geometry>
+				<mesh filename="${hokuyo_mesh_path}" />
+			</geometry>
+		</visual>
+	</link>
 	<joint name="base_robot_to_base_wheel" type="${wheel_kinematic_type}" >
 		<parent link="base_robot" />
@@ -73,3 +83,9 @@
 		<origin xyz="-${wheel_distance_x} -${wheel_distance_y} 0" />
 	</joint>
+	<joint name="base_robot_to_hokuyo" type="${wheel_kinematic_type}" >
+		<parent link="base_robot" />
+		<child link="hokuyo_laser" />
+		<axis xyz="0 1 0" />
+		<origin xyz="${wheel_distance_x} 0 0" />
+	</joint>
 </robot>

Commit message: upgrade

File: catkin/src/tutorials/testbot_description/urdf/robot_model.urdf.xacro (robot description, xacro)
@@ -5,8 +5,8 @@
 	<xacro:property name="wheel_distance_x" value="0.8"/>
 	<xacro:property name="wheel_distance_y" value="1" />
-	<xacro:property name="wheel_kinematic_type" value="fixed" />
+	<xacro:property name="wheel_kinematic_type" value="continuous" />
 	<xacro:property name="hokuyo_mesh_path" value="package://testbot_description/meshes/hokuyo.dae" />
 	<xacro:property name="hokuyo_kinematic_type" value="fixed" />
-	<link name="base_robot">
+	<link name="base_footprint">
 		<visual>
 			<origin rpy="0 0 0" xyz="0 0 0" />
@@ -51,5 +51,5 @@
 		</visual>
 	</link>
-	<link name="hokuyo_laser">
+	<link name="base_laser_link">
 		<visual>
 			<origin rpy="0 0 0" xyz="0 0 0" />
@@ -59,31 +59,31 @@
 		</visual>
 	</link>
-	<joint name="base_robot_to_base_wheel" type="${wheel_kinematic_type}" >
-		<parent link="base_robot" />
+	<joint name="base_footprint_to_base_wheel" type="${wheel_kinematic_type}" >
+		<parent link="base_footprint" />
 		<child link="base_wheel_back_left" />
 		<axis xyz="0 1 0" />
 		<origin xyz="-${wheel_distance_x} ${wheel_distance_y} 0" />
 	</joint>
-	<joint name="base_robot_to_base_wheel_front_right" type="${wheel_kinematic_type}" >
-		<parent link="base_robot" />
+	<joint name="base_footprint_to_base_wheel_front_right" type="${wheel_kinematic_type}" >
+		<parent link="base_footprint" />
 		<child link="base_wheel_front_right" />
 		<axis xyz="0 1 0" />
 		<origin xyz="${wheel_distance_x} -${wheel_distance_y} 0" />
 	</joint>
-	<joint name="base_robot_to_base_wheel_front_left" type="${wheel_kinematic_type}" >
-		<parent link="base_robot" />
+	<joint name="base_footprint_to_base_wheel_front_left" type="${wheel_kinematic_type}" >
+		<parent link="base_footprint" />
 		<child link="base_wheel_front_left" />
 		<axis xyz="0 1 0" />
 		<origin xyz="${wheel_distance_x} ${wheel_distance_y} 0" />
 	</joint>
-	<joint name="base_robot_to_base_wheel_back_right" type="${wheel_kinematic_type}" >
-		<parent link="base_robot" />
+	<joint name="base_footprint_to_base_wheel_back_right" type="${wheel_kinematic_type}" >
+		<parent link="base_footprint" />
 		<child link="base_wheel_back_right" />
 		<axis xyz="0 1 0" />
 		<origin xyz="-${wheel_distance_x} -${wheel_distance_y} 0" />
 	</joint>
-	<joint name="base_robot_to_hokuyo" type="${wheel_kinematic_type}" >
-		<parent link="base_robot" />
-		<child link="hokuyo_laser" />
+	<joint name="base_footprint_to_base_laser_link" type="${wheel_kinematic_type}" >
+		<parent link="base_footprint" />
+		<child link="base_laser_link" />
 		<axis xyz="0 1 0" />
 		<origin xyz="${wheel_distance_x} 0 0" />

Commit message: upgrade

File: catkin/src/tutorials/testbot_description/urdf/robot_model.urdf.xacro (robot description, xacro)
@@ -51,5 +51,5 @@
 		</visual>
 	</link>
-	<link name="base_laser_link">
+	<!-- <link name="base_laser_link">
 		<visual>
 			<origin rpy="0 0 0" xyz="0 0 0" />
@@ -58,5 +58,5 @@
 			</geometry>
 		</visual>
-	</link>
+	</link> -->
 	<joint name="base_footprint_to_base_wheel" type="${wheel_kinematic_type}" >
 		<parent link="base_footprint" />
@@ -83,9 +83,9 @@
 		<origin xyz="-${wheel_distance_x} -${wheel_distance_y} 0" />
 	</joint>
-	<joint name="base_footprint_to_base_laser_link" type="${wheel_kinematic_type}" >
+	<!-- <joint name="base_footprint_to_base_laser_link" type="${wheel_kinematic_type}" >
 		<parent link="base_footprint" />
 		<child link="base_laser_link" />
 		<axis xyz="0 1 0" />
 		<origin xyz="${wheel_distance_x} 0 0" />
-	</joint>
+	</joint> -->
 </robot>
