Commit message: upgrade

File: catkin/src/atwork_launch/urdf/atwork_model.urdf.xacro (robot description, xacro)
@@ -59,5 +59,17 @@
 		</visual>
 	</link> -->
-	<joint name="base_footprint_to_base_wheel" type="${wheel_kinematic_type}" >
+	<joint name="base_to_wheel_front_left" type="${wheel_kinematic_type}" >
+		<parent link="base_footprint" />
+		<child link="base_wheel_front_left" />
+		<axis xyz="0 1 0" />
+		<origin xyz="${wheel_distance_x} ${wheel_distance_y} 0" />
+	</joint>
+	<joint name="base_to_wheel_front_right" type="${wheel_kinematic_type}" >
+		<parent link="base_footprint" />
+		<child link="base_wheel_front_right" />
+		<axis xyz="0 1 0" />
+		<origin xyz="${wheel_distance_x} -${wheel_distance_y} 0" />
+	</joint>
+	<joint name="base_to_wheel_back_left" type="${wheel_kinematic_type}" >
 		<parent link="base_footprint" />
 		<child link="base_wheel_back_left" />
@@ -65,17 +77,5 @@
 		<origin xyz="-${wheel_distance_x} ${wheel_distance_y} 0" />
 	</joint>
-	<joint name="base_footprint_to_base_wheel_front_right" type="${wheel_kinematic_type}" >
-		<parent link="base_footprint" />
-		<child link="base_wheel_front_right" />
-		<axis xyz="0 1 0" />
-		<origin xyz="${wheel_distance_x} -${wheel_distance_y} 0" />
-	</joint>
-	<joint name="base_footprint_to_base_wheel_front_left" type="${wheel_kinematic_type}" >
-		<parent link="base_footprint" />
-		<child link="base_wheel_front_left" />
-		<axis xyz="0 1 0" />
-		<origin xyz="${wheel_distance_x} ${wheel_distance_y} 0" />
-	</joint>
-	<joint name="base_footprint_to_base_wheel_back_right" type="${wheel_kinematic_type}" >
+	<joint name="base_to_wheel_back_right" type="${wheel_kinematic_type}" >
 		<parent link="base_footprint" />
 		<child link="base_wheel_back_right" />

Commit message: upgrade

File: catkin/src/atwork_launch/urdf/atwork_model.urdf.xacro (robot description, xacro)
@@ -51,5 +51,5 @@
 		</visual>
 	</link>
-	<!-- <link name="base_laser_link">
+	<link name="base_laser_link">
 		<visual>
 			<origin rpy="0 0 0" xyz="0 0 0" />
@@ -58,5 +58,5 @@
 			</geometry>
 		</visual>
-	</link> -->
+	</link>
 	<joint name="base_to_wheel_front_left" type="${wheel_kinematic_type}" >
 		<parent link="base_footprint" />
@@ -83,9 +83,9 @@
 		<origin xyz="-${wheel_distance_x} -${wheel_distance_y} 0" />
 	</joint>
-	<!-- <joint name="base_footprint_to_base_laser_link" type="${wheel_kinematic_type}" >
+	<joint name="base_to_laser_link" type="${wheel_kinematic_type}" >
 		<parent link="base_footprint" />
 		<child link="base_laser_link" />
 		<axis xyz="0 1 0" />
 		<origin xyz="${wheel_distance_x} 0 0" />
-	</joint> -->
+	</joint>
 </robot>

Commit message: upgrade

File: catkin/src/atwork_launch/urdf/atwork_model.urdf.xacro (robot description, xacro)
@@ -51,5 +51,5 @@
 		</visual>
 	</link>
-	<link name="base_laser_link">
+	<link name="base_laser_link_node">
 		<visual>
 			<origin rpy="0 0 0" xyz="0 0 0" />
@@ -83,7 +83,7 @@
 		<origin xyz="-${wheel_distance_x} -${wheel_distance_y} 0" />
 	</joint>
-	<joint name="base_to_laser_link" type="${wheel_kinematic_type}" >
+	<joint name="base_to_laser_link_node" type="${wheel_kinematic_type}" >
 		<parent link="base_footprint" />
-		<child link="base_laser_link" />
+		<child link="base_laser_link_node" />
 		<axis xyz="0 1 0" />
 		<origin xyz="${wheel_distance_x} 0 0" />
